File: PolivoksVCF_panel.kicad_pcb (KiCad board)
At the start: 2 copper layers, 30 x 128.5 mm, 11 parts

Commit message: Added panel
Parts:
- added ?: LOGO, PolivoksVCF:Kraakenstuff, F.Cu at (38.9, 146.1)
- added ~: LOGO, PolivoksVCF:BP, F.Cu at (42.3, 88.1)
- added ~: LOGO, PolivoksVCF:Cutoff, F.Cu at (33.0, 43.4)
- added ~: LOGO, PolivoksVCF:VCF, F.Cu at (44.5, 28.2)
- added ~: LOGO, PolivoksVCF:Polivoks, F.Cu at (38.7, 25.1)
- added ~: LOGO, PolivoksVCF:LP, F.Cu at (23.7, 88.1)
- added ~: LOGO, PolivoksVCF:Out, F.Cu at (40.8, 136.8)
- added ~: LOGO, PolivoksVCF:In, F.Cu at (25.1, 135.9)
- added ~: LOGO, PolivoksVCF:CV2, F.Cu at (40.8, 122.8)
- added ~: LOGO, PolivoksVCF:CV1, F.Cu at (25.1, 122.8)
- added ~: LOGO, PolivoksVCF:Att2, F.Cu at (40.8, 107.7)
- added ~: LOGO, PolivoksVCF:Att1, F.Cu at (25.1, 107.7)
- added ~: LOGO, PolivoksVCF:Resonance, F.Cu at (33.1, 70.7)
Routing:
- net (no net): track 0.00 -> 3041.6 mm
Other:
- net class Default: trace_width 0.25 -> 0.5
